File: pinguino-2550-v2/pinguino-2550.sch (KiCad schematic (older format))
At the start: 25 parts, among them J1 USB, J10 D1, J11 D2, J12 D3, J2 BATT, J3 SELECT, J4 A0, J5 A1, J6 PWM-1, J8 UART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

Commit message: Added BoM. Fixed pcbnew paper size.
Other:
- note added: "Referencia\n==========\n| C1 100nF\n| C2 10uF\n| C3 22pF\n| C4 22pF\n| C5 220nF\n| D1 PWRLED\n| D2 USERLED\n| J1 USB (Conector USB tipo B)\n| J2 BATT (Bornera alimentación externa)\n| J3 SELECT (Jumper seleción alim. externa o USB)\n| J4 A0 (Bornera entradas analógicas)\n| J5 A1 (Bornera entradas analógicas)\n| J6 PWM-1 (Bornera salidas analógicas)\n| J8 UART (Bornera puerto serie)\n| J9 D0 (Born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"
Changed lines of the file:
@@
-EESchema Schematic File Version 2  date jue 03 abr 2014 00:37:07 ART
+EESchema Schematic File Version 2  date vie 04 abr 2014 20:51:02 ART
 LIBS:power
 LIBS:device
@@
 Sheet 1 1
 Title "Pinguino 2550"
-Date "2 apr 2014"
+Date "4 apr 2014"
 Rev "2.0.1"
 Comp "E.E.T. Nro.7 - Banfield"
@@
 Wire Wire Line
 	5700 9300 4950 9300
+Text Notes 600  8800 0    60   ~ 0
+Referencia\n==========\n| C1         100nF\n| C2         10uF\n| C3         22pF\n| C4         22pF\n| C5         220nF\n| D1         PWRLED\n| D2         USERLED\n| J1         USB (Conector USB tipo B)\n| J2         BATT (Bornera alimentación externa)\n| J3         SELECT (Jumper seleción alim. externa o USB)\n| J4         A0 (Bornera entradas analógicas)\n| J5         A1 (Bornera entradas analógicas)\n| J6         PWM-1 (Bornera salidas analógicas)\n| J8         UART (Bornera puerto serie)\n| J9         D0 (Bornera salidas digitales)\n| J10        D1 (Bornera salidas digitales)\n| J11        D2\n| J12        D3\n| R1         470\n| R2         10K\n| R3         470\n| SW1        RESET\n| U1         PIC18F2550\n| U2         LM7805CT\n| X1         20Mhz
 $EndSCHEMATC
